File: nx41-lm317.kicad_pcb (KiCad board)
At the start: 2 copper layers, 5 parts, among them J1 Conn_01x02, J2 Conn_01x02, U1 LM317_TO-220

Commit message: Platine
Other:
- board text added: "https://github.com/b-oern/nx41_lm317"
Changed lines of the file:
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@@
     )
+  )
+  (gr_text "https://github.com/b-oern/nx41_lm317" (at 75.71 68.7) (layer "B.SilkS")
+    (effects (font (size 1 1) (thickness 0.15)) (justify mirror))
   )
   (gr_text "GND" (at 68.18 66.09 90) (layer "F.SilkS")
