File: nx41-lm317.kicad_sch (KiCad schematic)
At the start: 5 parts, among them J1 Conn_01x02, J2 Conn_01x02, U1 LM317_TO-220

Commit message: Platine
Parts:
- C1: footprint (none) -> Capacitor_THT:CP_Radial_D5.0mm_P2.50mm
- J1, J2: footprint (none) -> TerminalBlock:TerminalBlock_bornier-2_P5.08mm
- R1: footprint (none) -> Resistor_THT:R_Axial_DIN0414_L11.9mm_D4.5mm_P5.08mm_Vertical
Changed lines of the file:
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@@
     (property "Reference" "R1" (id 0) (at 86.36 57.5142 90))
     (property "Value" "R" (id 1) (at 86.36 60.0511 90))
-    (property "Footprint" "" (id 2) (at 86.36 60.452 90)
+    (property "Footprint" "Resistor_THT:R_Axial_DIN0414_L11.9mm_D4.5mm_P5.08mm_Vertical" (id 2) (at 86.36 60.452 90)
       (effects (font (size 1.27 1.27)) hide)
     )
@@
       (effects (font (size 1.27 1.27)) (justify right))
     )
-    (property "Footprint" "" (id 2) (at 101.6 62.23 0)
+    (property "Footprint" "TerminalBlock:TerminalBlock_bornier-2_P5.08mm" (id 2) (at 101.6 62.23 0)
       (effects (font (size 1.27 1.27)) hide)
     )
@@
       (effects (font (size 1.27 1.27)) (justify left))
     )
-    (property "Footprint" "" (id 2) (at 59.3852 72.39 0)
+    (property "Footprint" "Capacitor_THT:CP_Radial_D5.0mm_P2.50mm" (id 2) (at 59.3852 72.39 0)
       (effects (font (size 1.27 1.27)) hide)
     )
@@
     (property "Reference" "J1" (id 0) (at 45.085 58.454 0))
     (property "Value" "Conn_01x02" (id 1) (at 46.99 66.04 0))
-    (property "Footprint" "" (id 2) (at 44.45 62.23 0)
+    (property "Footprint" "TerminalBlock:TerminalBlock_bornier-2_P5.08mm" (id 2) (at 44.45 62.23 0)
       (effects (font (size 1.27 1.27)) hide)
     )
@@
     )
     (path "/8a79efce-e090-47e5-b400-55929c6b84ce"
-      (reference "C1") (unit 1) (value "C") (footprint "")
+      (reference "C1") (unit 1) (value "C") (footprint "Capacitor_THT:CP_Radial_D5.0mm_P2.50mm")
     )
     (path "/cac095cf-1a8d-4a4d-a616-f3dfff74bd9a"
-      (reference "J1") (unit 1) (value "Conn_01x02") (footprint "")
+      (reference "J1") (unit 1) (value "Conn_01x02") (footprint "TerminalBlock:TerminalBlock_bornier-2_P5.08mm")
     )
     (path "/74fe512a-302b-4d3c-a57e-7dccec2ce4d3"
-      (reference "J2") (unit 1) (value "Conn_01x02") (footprint "")
+      (reference "J2") (unit 1) (value "Conn_01x02") (footprint "TerminalBlock:TerminalBlock_bornier-2_P5.08mm")
     )
     (path "/60a0dc87-ccb5-4848-93d9-de1ed482c789"
-      (reference "R1") (unit 1) (value "R") (footprint "")
+      (reference "R1") (unit 1) (value "R") (footprint "Resistor_THT:R_Axial_DIN0414_L11.9mm_D4.5mm_P5.08mm_Vertical")
     )
     (path "/7a9a8cd0-c365-45db-997a-4ad21211684f"
